File: powersupply.brd (EAGLE design)
At the start: 100 x 80 mm, 33 parts, among them IC1 LM1117MPX-3.3, IC2 STM32F030F4P, Q1 IRF7425, Q2 BSS138, Q3 IRF7425, Q4 BSS138, Q5 IRF7425, Q6 BSS138, Q7 IRF7425, Q8 BSS138, X1 53261-04

Commit message: йй
Parts:
- removed Q4, Q6: BSS138, m-pad-2.1:SOT23
- removed Q5: IRF7425, m-pad-2.1:SO-8
- added C11, C14: 22uF, rcl:C0805
- added C12, C7: 4.7uF, rcl:C0805
- added C13, C15, C18, C4, C5, C8: 0.1uF, rcl:C0805
- added C16, C17, C19, C20, C21, C3: 10uF, rcl:C0805
- added GPIO1, GPIO2, GPIO3, GPIO5, GPIO6: WIREPAD1,6/0,9, wirepad:1,6/0,9
- added IC4, IC5: ST1S10PHR, vreg-pulse:HSOP8
- added L1: (no value), inductor-neosid:SM-1206
- added L3, L4: BCIHP0730-3R3M, m-pad-2.1:INDUCTOR_SLF7045
- added PAD6, PAD7, PAD8: WIREPAD2,54/0,9, wirepad:2,54/0,9
- added R13: 680, rcl:M0805
- added R14: 10K, rcl:M0805
- added R15: 100K, rcl:M0805
- added R16, R18, R19: 20K, rcl:M0805
- added R17: 105K, rcl:M0805
- added U$1: GL852G-SSOP28, genesys-logic:SSOP28
- added Z2, Z3: NFE31PT, emi-filter:NFE31
- Q3: value IRF7425 -> (none); device m-pad-2.1:SO-8 -> crystal-geyer_V1_0:6.0X3.5_2
- R5: value (none) -> 100K; device resistor:R0805 -> rcl:M0805
- R6: value (none) -> 20K; device resistor:R0805 -> rcl:M0805
- R7: value (none) -> 10K; device resistor:R0805 -> rcl:M0805
- R8: value (none) -> 105K; device resistor:R0805 -> rcl:M0805
- moved R8 184.5 mm to (113.7, 39.2), turned to 270 degrees
- moved R6 158.5 mm to (106.3, 31.5), turned to 270 degrees
- moved R7 120.1 mm to (4.95, 29.7), turned to 180 degrees
- moved R5 92.6 mm to (4.95, 27.3), turned to 180 degrees
- moved Q3 79.4 mm to (13.5, 19.1)
- moved C10 36.9 mm to (69.6, 7.11)
- moved C6 36.9 mm to (74.5, 10.2)
- moved C9 36.9 mm to (68.6, 19.1)
- moved IC2 36.9 mm to (68.6, 12.7)
- moved R11 36.9 mm to (74.5, 14.5)
- moved R12 36.9 mm to (65.7, 5.71)
- moved S2 36.9 mm to (77.7, 12.3)
- moved X1 36.9 mm to (67.3, 33.0)
Connections:
- removed net +5V1: Q5.3, R6.2
- removed net POWER_MONITOR: Q4.1, R7.2
- removed net POWER_PC: Q6.1, R8.2
- removed net ПИТАНИЕ_МОНИТОРА: Q3.8
- new net +5V: GPIO1.1
- new net DM: GPIO3.1, U$1.25
- new net DP: GPIO5.1, U$1.26
- new net EN_IN: IC4.2, IC5.2, R18.2, R19.2
- new net GND2: C11.1, C7.1, C8.1, IC4.4, IC4.5, IC4.8, IC4.H@1, IC4.H@2, IC4.H@3, IC4.H@4, IC4.H@5, IC4.H@6, R16.2, R18.1, Z2.2
- new net GND3: C12.1, C13.1, C14.1, IC5.4, IC5.5, IC5.8, IC5.H@1, IC5.H@2, IC5.H@3, IC5.H@4, IC5.H@5, IC5.H@6, R19.1, R6.2, Z3.2
- new net N$10: IC4.7, L3.1
- new net N$11: C11.2, L3.2, R17.1, Z2.1
- new net N$13: IC4.3, R16.1, R17.2
- new net N$14: C14.2, L4.2, R8.1, Z3.1
- new net N$15: IC5.3, R6.1, R8.2
- new net N$16: R13.1, U$1.4
- new net N$17: C19.2, R14.1, R15.2, U$1.13
- new net N$18: C21.2, Q3.1, U$1.7
- new net N$19: C20.2, Q3.2, U$1.6
- new net N$5: C15.1, C16.1, C5.1, L1.2, U$1.1, U$1.10, U$1.5
- new net N$6: R7.1, U$1.17
- new net N$8: R5.1, U$1.18
- new net VBUS: C17.2, C18.2, GPIO2.1, R14.2, U$1.23
- net +12VBATT: now also C12.2, C13.2, C7.2, C8.2, IC4.1, IC4.6, IC5.1, IC5.6; no longer Q3.3, R5.2
- net GND: now also C15.2, C16.2, C17.1, C18.1, C19.1, C20.1, C21.1, C3.1, C4.1, C5.2, GPIO6.1, R13.2, R15.1; no longer Q4.2, Q6.2, R7.1, R8.1
- net N$12: now also IC5.7, L4.1; no longer Q5.4, Q6.3, R6.1
- net N$9: now also C3.2, C4.2, L1.1, R5.2, R7.2, U$1.16, U$1.24; no longer Q3.4, Q4.3, R5.1
- net ПИТАНИЕ_ПК: now also Z2.3; no longer Q5.8
- net ПИТАНИЕ_ХАБ: now also Z3.3; no longer Q7.8
Routing:
- net +12VBATT: track 0.00 -> 72.3 mm
- net N$5: track 0.00 -> 16.6 mm, vias 0 -> 2
- net N$18: track 0.00 -> 14.4 mm
- net N$9: track 0.00 -> 14.1 mm, vias 0 -> 2
- net N$19: track 0.00 -> 13.6 mm
- net N$15: track 0.00 -> 13.4 mm, vias 0 -> 2
- net N$13: track 0.00 -> 13.4 mm, vias 0 -> 2
- net EN_IN: track 0.00 -> 13.2 mm
- net N$14: track 0.00 -> 10.7 mm
- net N$11: track 0.00 -> 10.7 mm
- net N$17: track 0.00 -> 9.58 mm
- net VBUS: track 0.00 -> 6.39 mm
- net N$12: track 0.00 -> 5.71 mm
- net N$10: track 0.00 -> 5.71 mm
- net N$8: track 0.00 -> 4.51 mm
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- added copper zone on layer 1, net GND
- added copper zone on layer 1, net GND2
- added copper zone on layer 1, net GND3
Other:
- board size 100 x 80 mm -> 81.9 x 55.9 mm

Commit message: 1
Parts:
- removed C10, C6, C9: 0.1uf, rcl:C0805
- removed C13: 0.1uF, rcl:C0805
- removed C20, C21: 10uF, rcl:C0805
- removed C7: 4.7uF, rcl:C0805
- removed GPIO1, GPIO2, GPIO3, GPIO5, GPIO6: WIREPAD1,6/0,9, wirepad:1,6/0,9
- removed IC5: ST1S10PHR, vreg-pulse:HSOP8
- removed L1: (no value), inductor-neosid:SM-1206
- removed L3, L4: BCIHP0730-3R3M, m-pad-2.1:INDUCTOR_SLF7045
- removed PAD6, PAD7, PAD8: WIREPAD2,54/0,9, wirepad:2,54/0,9
- removed Q2, Q8: BSS138, m-pad-2.1:SOT23
- removed Q3: (no value), crystal-geyer_V1_0:6.0X3.5_2
- removed Q7: IRF7425, m-pad-2.1:SO-8
- removed R11, R12: 10K, rcl:M0805
- removed R16, R18, R19: 20K, rcl:M0805
- removed R17: 105K, rcl:M0805
- removed X1: 53261-04, con-molex:53261-04
- removed Z2, Z3: NFE31PT, emi-filter:NFE31
- added +12VSCR\, +5V, +5VHUB, 22, 23, 28, 29, 30, 31, 32, 3V3_1, DM1, DP1, GND, GNDGPS, GNDHUB, GNDSCR, GPIO27, PWR_BT+, PWR_BT-, RTC+, RTC-, RX, TX: (no value), wirepad:1,6/0,8
- added 1WIRE: (no value), con-molex:53047-03
- added BT1: CH291-1220LF, battery:CH291-1220LF
- added BTN: 53047-03, con-molex:53047-03
- added F1, F3: 6V/0.5A, SparkFun-Fuses:1206
- added F2: 6V 0.5A, SparkFun-Fuses:0805
- added FAN2: 53047-02, con-molex:53047-02
- added GPS, I2C_VIM, SWD, USB1: 53047-04, con-molex:53047-04
- added I2C, PC_PWR: i2c, con-molex:53047-04
- added I2SVIM: 53047-06, con-molex:53047-06
- added L2: BCIHP0730-3R3M, bt_inductor:VLS4045EX
- added PWR: JST-XH-03-PIN-ROUND-PAD, Rembrandt Electronics - JST XH Connectors v1-0:JST-XH-03-PACKAGE-ROUND-PAD
- added U2: TPS54428, borkedlabs-powerics:PDSO-8
- C1, C2: value (none) -> 0.1uf
- C11: value 22uF -> 0.1uf
- C12: value 4.7uF -> 0.1uf
- C14: value 22uF -> 0.1uF; device rcl:C0805 -> rcl:C0805K
- C15: value 0.1uF -> 22uF
- C16: value 10uF -> 1uF; device rcl:C0805 -> rcl:C0805K
- C17: value 10uF -> 8.2nF; device rcl:C0805 -> rcl:C0805K
- C18: device rcl:C0805 -> rcl:C0805K
- C19: value 10uF -> 47uF; device rcl:C0805 -> rcl:C1206
- C3: value 10uF -> (none); device rcl:C0805 -> rcl:UD-8X10_NICHICON
- C4: value 0.1uF -> (none); device rcl:C0805 -> rcl:UD-8X10_NICHICON
- C5: value 0.1uF -> 47uF; device rcl:C0805 -> rcl:C1206
- C8: value 0.1uF -> 0.1uf
- D1: device diode:SOD323-W -> diode:SMB
- IC2: value STM32F030F4P -> BTS716G; device micro-stm_v3:TSSOP20-I -> infineon:PG-DSO-20
- IC4: value ST1S10PHR -> STM32F030F4P; device vreg-pulse:HSOP8 -> micro-stm_v3:TSSOP20-I
- OC1: value PC817 -> PC817SMD; device my_mixed:DIL04 -> my_mixed:DIL04SMD
- Q1: value IRF7425 -> BSS138; device m-pad-2.1:SO-8 -> m-pad-2.1:SOT23
- R1, R10, R2: value (none) -> 150
- R13: value 680 -> 22.1K
- R14: value 10K -> 124K
- R15: value 100K -> 10k
- R3: value (none) -> 10k
- R4: value (none) -> 2.2k
- R5: value 100K -> 10k; device rcl:M0805 -> resistor:R0805
- R6: value 20K -> 10k; device rcl:M0805 -> resistor:R0805
- R8: value 105K -> 10K
- R9: value (none) -> 10K; device resistor:R0805 -> rcl:M0805
- U$1: value GL852G-SSOP28 -> MP1584; device genesys-logic:SSOP28 -> MP1584-dc-brick:DC-BRICK
- moved R9 181.1 mm to (16.5, 40.6)
- moved R10 155.7 mm to (23.5, 22.6), turned to 180 degrees
- moved C2 152.2 mm to (26.7, 29.2), turned to 90 degrees
- moved C1 148.4 mm to (29.2, 29.2), turned to 90 degrees
- moved IC1 145.5 mm to (26.2, 36.3)
- moved OC1 134.3 mm to (8.89, 41.9), turned to 90 degrees
- moved R4 110.8 mm to (69.5, 22.0), flipped to the bottom
- moved C11 110.7 mm to (10.2, 29.2)
- moved C14 108.0 mm to (10.7, 17.9), turned to 180 degrees
- moved R3 106.1 mm to (69.5, 19.7), flipped to the bottom, turned to 180 degrees
- moved IC4 99.8 mm to (16.5, 27.9), turned to 90 degrees
- moved C12 97.0 mm to (22.1, 29.0), turned to 90 degrees
- moved D2 92.1 mm to (65.8, 20.6), flipped to the bottom, turned to 90 degrees
- moved R8 91.3 mm to (23.5, 25.0), turned to 180 degrees
- moved C8 91.2 mm to (19.1, 33.9), turned to 0 degrees
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Connections:
- removed net +12VACC: D3.C, Q2.1, R2.2, R3.1, R4.2
- removed net +12VBATT: C12.2, C13.2, C7.2, C8.2, IC4.1, IC4.6, IC5.1, IC5.6, Q1.8
- removed net +5V: GPIO1.1
- removed net +5V2: Q7.3, R9.2
- removed net +BATT: D1.A
- removed net DM: GPIO3.1, U$1.25
- removed net DP: GPIO5.1, U$1.26
- removed net EN_IN: IC4.2, IC5.2, R18.2, R19.2
- removed net GND2: C11.1, C7.1, C8.1, IC4.4, IC4.5, IC4.8, IC4.H@1, IC4.H@2, IC4.H@3, IC4.H@4, IC4.H@5, IC4.H@6, R16.2, R18.1, Z2.2
- removed net GND3: C12.1, C13.1, C14.1, IC5.4, IC5.5, IC5.8, IC5.H@1, IC5.H@2, IC5.H@3, IC5.H@4, IC5.H@5, IC5.H@6, R19.1, R6.2, Z3.2
- removed net N$17: C19.2, R14.1, R15.2, U$1.13
- removed net POWER_HUB: Q8.1, R10.2
- removed net VBUS: C17.2, C18.2, GPIO2.1, R14.2, U$1.23
- removed net ПИТАНИЕ_ПК: Z2.3
- removed net ПИТАНИЕ_ХАБ: Z3.3
- new net 1WIRE: 1WIRE.1, IC4.11
- new net 3V3: 3V3_1.1, GPIO27.1, GPS.4, I2C_VIM.4, I2SVIM.6, IC4.7
- new net ACC: D2.A, IC4.8, R3.1, R4.2
- new net ARDUINO_PWR: C1.2, IC1.3, IC2.18
- new net BCK: 30.1, I2SVIM.3
- new net FAN: IC4.13, R10.2
- new net HUB_CTRL: IC2.9, IC4.9
- new net HUB_PWR: IC2.13, U$1.IN1+, U$1.IN2+
- new net I2C_SCK_A: 22.1, I2C_VIM.2
- new net I2C_SDA_A: 23.1, I2C_VIM.3
- new net I2S_LCK: 32.1, I2SVIM.5
- new net I2S_SCK: 29.1, I2SVIM.2
- new net I2S_SDO: 31.1, I2SVIM.4
- new net N$23: +12VSCR\.1, F3.2
- new net N$51: C16.2, U2.4
- new net N$52: C17.2, U2.3
- new net N$53: C18.1, U2.7
- new net N$54: C18.2, L2.1, U2.6
- new net N$55: R13.1, R14.2, U2.2
- new net N$56: R15.2, U2.1
- new net PC_CTRL: IC2.7, IC4.2
- new net PC_PWR: C14.1, C15.2, IC2.14, R15.1, U2.8
- new net SCL: I2C.3, IC4.17
- new net SCREEN_CTRL: IC2.5, IC4.3
- new net SCREEN_PWR: F3.1, IC2.17
- new net SDA: I2C.2, IC4.18
- new net VBB: C3.+, C4.+, F1.2, IC2.1, IC2.10, IC2.11, IC2.12, IC2.15, IC2.16, IC2.19, IC2.20
- new net VIM_BTN: IC4.12, R9.2
- new net VIM_PWR_CTRL: OC1.1, R9.1
- new net VOUT5V: C19.2, C5.2, FAN2.1, L2.2, PC_PWR.1, PC_PWR.2, R13.2
- net +ACC: now also F2.2, R3.2; no longer D2.A
- net BOOT0: now also IC4.1, R8.2; no longer IC2.1, R12.2
- net GND: now also 1WIRE.2, 28.1, C11.2, C12.2, C14.2, C15.1, C16.1, C3.-, C4.-, C5.1, C8.2, GND.1, GNDGPS.1, GNDHUB.1, GNDSCR.1, GPS.1, I2C.4, I2C_VIM.1, I2SVIM.1, IC4.15, OC1.2, PC_PWR.3, PC_PWR.4, PWR.2, Q1.2, R1.2, R14.1, R2.2, R5.2, R6.2, R8.1, SWD.4, U$1.IN1-, U$1.IN2-, U$1.OUT1-, U$1.OUT2-, U2.5, U2.PAD, USB1.4; no longer C10.2, C15.2, C16.2, C18.1, C20.1, C21.1, C3.1, C4.1, C5.2, C6.2, C9.2, GPIO6.1, IC2.15, Q2.2, Q8.2, R10.1, R12.1, R13.2, R15.1, R2.1, X1.4
- net N$1: now also IC2.2, R1.1; no longer D1.C, Q1.3, R1.2
- net N$10: now also BT1.-, RTC-.1; no longer IC4.7, L3.1
- net N$11: now also GPS.2, RX.1; no longer C11.2, L3.2, R17.1, Z2.1
- net N$12: now also GPS.3, TX.1; no longer IC5.7, L4.1
- net N$13: now also BTN.2, IC4.6, R5.1; no longer IC4.3, R16.1, R17.2
- net N$14: now also F2.1, PWR.3; no longer C14.2, L4.2, R8.1, Z3.1
- net N$15: now also BT1.+, RTC+.1; no longer IC5.3, R6.1, R8.2
- net N$16: now also D1.A, PWR.1; no longer R13.1, U$1.4
- net N$18: now also +5VHUB.1, U$1.OUT1+, U$1.OUT2+; no longer C21.2, Q3.1, U$1.7
- net N$19: now also D1.C, F1.1; no longer C20.2, Q3.2, U$1.6
- net N$2: now also +5V.1, USB1.1; no longer D2.C, R3.2
- net N$3: now also FAN2.2, Q1.3; no longer Q7.4, Q8.3, R9.1
- net N$4: now also D2.C, D3.C, IC2.3; no longer Q1.4, Q2.3, R1.1
- net N$5: now also IC2.6, R2.1; no longer C15.1, C16.1, C5.1, L1.2, U$1.1, U$1.10, U$1.5
- net N$6: now also BTN.1, IC4.10, R6.1; no longer R7.1, U$1.17
- net N$7: now also DM1.1, USB1.2; no longer C1.2, IC1.3
- net N$8: now also DP1.1, USB1.3; no longer R5.1, U$1.18
- net N$9: now also Q1.1, R10.1; no longer C3.2, C4.2, L1.1, R5.2, R7.2, U$1.16, U$1.24
- net NRST: now also C8.1, IC4.4, R7.1; no longer C6.1, IC2.4, R11.1
- net SELF_POWER: now also IC4.14
- net SWCLK: now also IC4.20, SWD.3; no longer IC2.20, X1.3
- net SWIO: now also IC4.19, SWD.2; no longer IC2.19, X1.2
- net VDD: now also 1WIRE.3, BTN.3, C11.1, C12.1, I2C.1, IC1.TAB, IC4.16, IC4.5, R7.2, SWD.1; no longer C10.1, C9.1, IC2.16, IC2.5, R11.2, X1.1
- net VIM_POWER+: now also OC1.3, PWR_BT+.1; no longer OC1.4
- net VIM_POWER-: now also OC1.4, PWR_BT-.1; no longer OC1.3
Routing:
- net VBB: track 0.00 -> 76.5 mm
- net SCREEN_CTRL: track 0.00 -> 73.5 mm, vias 0 -> 2
- net +12VBATT: track 72.3 -> 0.00 mm
- net N$4: track 0.00 -> 69.4 mm, vias 0 -> 3
- net HUB_CTRL: track 0.00 -> 63.7 mm, vias 0 -> 2
- net VDD: track 6.61 -> 69.0 mm, vias 0 -> 22
- net VOUT5V: track 0.00 -> 59.9 mm
- net 3V3: track 0.00 -> 59.6 mm
- net PC_CTRL: track 0.00 -> 58.0 mm, vias 0 -> 2
- net PC_PWR: track 0.00 -> 57.1 mm, vias 0 -> 2
- net ACC: track 0.00 -> 55.8 mm, vias 0 -> 1
- net SCREEN_PWR: track 0.00 -> 49.4 mm, vias 0 -> 1
- net I2S_SCK: track 0.00 -> 41.8 mm
- net ARDUINO_PWR: track 0.00 -> 41.0 mm
- net BCK: track 0.00 -> 40.0 mm
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- added copper zone on layer 16, net GND
- added copper zone on layer 1, net N$54
- added copper zone on layer 1, net PC_PWR
- added copper zone on layer 1, net VBB
- added copper zone on layer 1, net VDD
- added copper zone on layer 16, net VDD
- removed copper zone on layer 1, net GND2
- removed copper zone on layer 1, net GND3
- removed copper zone on layer 1, net NC2
- removed copper zone on layer 16, net NC3

Commit message: фиксы схемы
R9 FROM 10K TO 120Ohm
SWAP R13 and R14 nominal
Parts:
- R13: value 22.1K -> 124K
- R14: value 124K -> 22.1К
- R9: value 10K -> 120
Changed lines of the file:
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@@
 <attribute name="VALUE" x="22.8" y="14.14" size="0.0254" layer="27"/>
 </element>
-<element name="R9" library="rcl" library_urn="urn:adsk.eagle:library:334" package="M0805" package3d_urn="urn:adsk.eagle:package:23556/2" value="10K" x="16.51" y="40.64" smashed="yes">
+<element name="R9" library="rcl" library_urn="urn:adsk.eagle:library:334" package="M0805" package3d_urn="urn:adsk.eagle:package:23556/2" value="120" x="16.51" y="40.64" smashed="yes">
 <attribute name="SPICEPREFIX" value="R" x="16.51" y="40.64" size="1.778" layer="27" display="off"/>
 <attribute name="VALUE" x="15.24" y="41.91" size="1.016" layer="27"/>
@@
 <attribute name="VALUE" x="15.612" y="2.935" size="1.016" layer="27"/>
 </element>
-<element name="R13" library="rcl" library_urn="urn:adsk.eagle:library:334" package="M0805" package3d_urn="urn:adsk.eagle:package:23556/2" value="22.1K" x="3.757" y="17.413" smashed="yes" rot="R90">
+<element name="R13" library="rcl" library_urn="urn:adsk.eagle:library:334" package="M0805" package3d_urn="urn:adsk.eagle:package:23556/2" value="124K" x="3.757" y="17.413" smashed="yes" rot="R90">
 <attribute name="MPN" value="TR0805B22K1P0525Z" x="3.757" y="17.413" size="1.778" layer="27" rot="R90" display="off"/>
 <attribute name="SPICEPREFIX" value="R" x="-2.593" y="17.413" size="1.778" layer="27" rot="R90" display="off"/>
 <attribute name="VALUE" x="1.763" y="19.917" size="1.016" layer="27" rot="R270"/>
 </element>
-<element name="R14" library="rcl" library_urn="urn:adsk.eagle:library:334" package="M0805" package3d_urn="urn:adsk.eagle:package:23556/2" value="124K" x="2.831" y="13.481" smashed="yes">
+<element name="R14" library="rcl" library_urn="urn:adsk.eagle:library:334" package="M0805" package3d_urn="urn:adsk.eagle:package:23556/2" value="22.1К" x="2.831" y="13.481" smashed="yes">
 <attribute name="MPN" value="AR05BTCW1253" x="2.831" y="13.481" size="1.778" layer="27" display="off"/>
 <attribute name="SPICEPREFIX" value="R" x="2.831" y="7.131" size="1.778" layer="27" display="off"/>
