File: powersupply.sch (EAGLE design)
At the start: 33 parts, among them IC1 LM1117MPX-3.3, IC2 STM32F030F4P, Q1 IRF7425, Q2 BSS138, Q3 IRF7425, Q4 BSS138, Q5 IRF7425, Q6 BSS138, Q7 IRF7425, Q8 BSS138, X1 53261-04

Commit message: йй
Parts:
- removed Q4, Q6: BSS138, m-pad-2.1:BSS138
- removed Q5: IRF7425, m-pad-2.1:IRF7425
- added C11, C14: 22uF, rcl:C-EUC0805
- added C12, C7: 4.7uF, rcl:C-EUC0805
- added C13, C15, C18, C4, C5, C8: 0.1uF, rcl:C-EUC0805
- added C16, C17, C19, C20, C21, C3: 10uF, rcl:C-EUC0805
- added GPIO1, GPIO2, GPIO3, GPIO5, GPIO6: WIREPAD1,6/0,9, wirepad:WIREPAD1,6/0,9
- added IC4, IC5: ST1S10PHR, vreg-pulse:ST1S10PHR
- added L1: (no value), inductor-neosid:SM-1206
- added L3, L4: BCIHP0730-3R3M, m-pad-2.1:L_EUH
- added PAD6, PAD7, PAD8: WIREPAD2,54/0,9, wirepad:WIREPAD2,54/0,9
- added R13: 680, rcl:R-EU_M0805
- added R14: 10K, rcl:R-EU_M0805
- added R15: 100K, rcl:R-EU_M0805
- added R16, R18, R19: 20K, rcl:R-EU_M0805
- added R17: 105K, rcl:R-EU_M0805
- added U$1: GL852G-SSOP28, genesys-logic:GL852G-SSOP28
- added Z2, Z3: NFE31PT, emi-filter:NFE31PT
- Q3: value IRF7425 -> (none); device m-pad-2.1:IRF7425 -> crystal-geyer_V1_0:KX-12B
- R5: value (none) -> 100K; device resistor:R-EU_R0805 -> rcl:R-EU_M0805
- R6: value (none) -> 20K; device resistor:R-EU_R0805 -> rcl:R-EU_M0805
- R7: value (none) -> 10K; device resistor:R-EU_R0805 -> rcl:R-EU_M0805
- R8: value (none) -> 105K; device resistor:R-EU_R0805 -> rcl:R-EU_M0805
Connections:
- removed net +5V1: Q5.S@3, R6.2
- removed net POWER_MONITOR: Q4.G, R7.2
- removed net POWER_PC: Q6.G, R8.2
- removed net ПИТАНИЕ_МОНИТОРА: Q3.D@4
- new net +5V: GPIO1.P
- new net DM: GPIO3.P, U$1.DM0
- new net DP: GPIO5.P, U$1.DP0
- new net EN_IN: IC4.EN, IC5.EN, R18.2, R19.2
- new net GND2: C11.1, C7.1, C8.1, IC4.AGND, IC4.H@1, IC4.H@2, IC4.H@3, IC4.H@4, IC4.H@5, IC4.H@6, IC4.PGND, IC4.SYNC, R16.2, R18.1, Z2.2
- new net GND3: C12.1, C13.1, C14.1, IC5.AGND, IC5.H@1, IC5.H@2, IC5.H@3, IC5.H@4, IC5.H@5, IC5.H@6, IC5.PGND, IC5.SYNC, R19.1, R6.2, Z3.2
- new net N$10: IC4.SW, L3.1
- new net N$11: C11.2, L3.2, R17.1, Z2.1
- new net N$13: IC4.FB, R16.1, R17.2
- new net N$14: C14.2, L4.2, R8.1, Z3.1
- new net N$15: IC5.FB, R6.1, R8.2
- new net N$16: R13.1, U$1.RREF
- new net N$17: C19.2, R14.1, R15.2, U$1.!RESET
- new net N$18: C21.2, Q3.1, U$1.X2
- new net N$19: C20.2, Q3.2, U$1.X1
- new net N$5: C15.1, C16.1, C5.1, L1.2, U$1.AVDD
- new net N$6: R7.1, U$1.PSELF
- new net N$8: R5.1, U$1.PGANG
- new net VBUS: C17.2, C18.2, GPIO2.P, R14.2, U$1.V5
- net +12VBATT: now also C12.2, C13.2, C7.2, C8.2, IC4.VIN_A, IC4.VIN_SW, IC5.VIN_A, IC5.VIN_SW; no longer Q3.S@3, R5.2
- net GND: now also C15.2, C16.2, C17.1, C18.1, C19.1, C20.1, C21.1, C3.1, C4.1, C5.2, GPIO6.P, R13.2, R15.1; no longer Q4.S, Q6.S, R7.1, R8.1
- net N$12: now also IC5.SW, L4.1; no longer Q5.G, Q6.D, R6.1
- net N$9: now also C3.2, C4.2, L1.1, R5.2, R7.2, U$1.DVDD, U$1.V33; no longer Q3.G, Q4.D, R5.1
- net ПИТАНИЕ_ПК: now also Z2.3; no longer Q5.D@4
- net ПИТАНИЕ_ХАБ: now also Z3.3; no longer Q7.D@4
Other:
- note added: "R1 = R2 x (VOUT - VFB) / VFB"
- moved on the sheet: C1, C2, D2, IC1, OC1, Q7, Q8, R10, R3, R4, R5, R6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

Commit message: 1
Parts:
- removed C10, C6, C9: 0.1uf, rcl:C-EUC0805
- removed C13: 0.1uF, rcl:C-EUC0805
- removed C20, C21: 10uF, rcl:C-EUC0805
- removed C7: 4.7uF, rcl:C-EUC0805
- removed GPIO1, GPIO2, GPIO3, GPIO5, GPIO6: WIREPAD1,6/0,9, wirepad:WIREPAD1,6/0,9
- removed IC5: ST1S10PHR, vreg-pulse:ST1S10PHR
- removed L1: (no value), inductor-neosid:SM-1206
- removed L3, L4: BCIHP0730-3R3M, m-pad-2.1:L_EUH
- removed PAD6, PAD7, PAD8: WIREPAD2,54/0,9, wirepad:WIREPAD2,54/0,9
- removed Q2, Q8: BSS138, m-pad-2.1:BSS138
- removed Q3: (no value), crystal-geyer_V1_0:KX-12B
- removed Q7: IRF7425, m-pad-2.1:IRF7425
- removed R11, R12: 10K, rcl:R-EU_M0805
- removed R16, R18, R19: 20K, rcl:R-EU_M0805
- removed R17: 105K, rcl:R-EU_M0805
- removed X1: 53261-04, con-molex:53261-04
- removed Z2, Z3: NFE31PT, emi-filter:NFE31PT
- added +12VSCR\, +5V, +5VHUB, 22, 23, 28, 29, 30, 31, 32, 3V3_1, DM1, DP1, GND, GNDGPS, GNDHUB, GNDSCR, GPIO27, PWR_BT+, PWR_BT-, RTC+, RTC-, RX, TX: (no value), wirepad:1,6/0,8
- added 1WIRE, BTN: 53047-03, con-molex:53047-03
- added BT1: CH291-1220LF, battery:CH291-1220LF
- added F1, F3: 6V/0.5A, SparkFun-Fuses:PPTC_HALF-AMP
- added F2: 6V 0.5A, SparkFun-Fuses:PPTC_6V500MA
- added FAN2: 53047-02, con-molex:53047-02
- added GPS, I2C_VIM, SWD, USB1: 53047-04, con-molex:53047-04
- added I2C, PC_PWR: i2c, con-molex:53047-04
- added I2SVIM: 53047-06, con-molex:53047-06
- added L2: BCIHP0730-3R3M, bt_inductor:VLS5045EX
- added PWR: JST-XH-03-PIN-ROUND-PAD, Rembrandt Electronics - JST XH Connectors v1-0:JST-XH-03-PIN-ROUND-PAD
- added U2: TPS54428, borkedlabs-powerics:TPS54428
- C1, C2: value (none) -> 0.1uf; MPN (none) -> CL21B104KBFNNNE
- C11: value 22uF -> 0.1uf; MPN (none) -> CL21B104KBFNNNE
- C12: value 4.7uF -> 0.1uf; MPN (none) -> CL21B104KBFNNNE
- C14: value 22uF -> 0.1uF; device rcl:C-EUC0805 -> rcl:C-EUC0805K; MPN (none) -> CL21B104KBFNNNE
- C15: value 0.1uF -> 22uF; MPN (none) -> CL31A226KAHNNNE; URL (none) -> https://lcsc.com/product-detail/Multilayer-Ceramic-Capacito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
- C16: value 10uF -> 1uF; device rcl:C-EUC0805 -> rcl:C-EUC0805K; MPN (none) -> CL21B105KAFNNNE; URL (none) -> https://lcsc.com/product-detail/Multilayer-Ceramic-Capacito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
- C17: value 10uF -> 8.2nF; device rcl:C-EUC0805 -> rcl:C-EUC0805K; MPN (none) -> CL21B822KBANNNC; URL (none) -> https://lcsc.com/product-detail/Multilayer-Ceramic-Capacito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
- C18: device rcl:C-EUC0805 -> rcl:C-EUC0805K; MPN (none) -> CL21B104KBFNNNE
- C19: value 10uF -> 47uF; device rcl:C-EUC0805 -> rcl:C-EUC1206; MPN (none) -> CL31A476MPHNNNE
- C3: value 10uF -> (none); device rcl:C-EUC0805 -> rcl:CPOL-EUUD-8X10
- C4: value 0.1uF -> (none); device rcl:C-EUC0805 -> rcl:CPOL-EUUD-8X10
- C5: value 0.1uF -> 47uF; device rcl:C-EUC0805 -> rcl:C-EUC1206; MPN (none) -> CL31A476MPHNNNE
- C8: value 0.1uF -> 0.1uf; MPN (none) -> CL21B104KBFNNNE
- D1: device diode:DIODE-SOD323-W -> diode:DIODE-SMB
- IC1: MPN (none) -> LM1117IMPX-3.3/NOPB
- IC2: value STM32F030F4P -> BTS716G; device micro-stm_v3:STM32F030F4P -> infineon:BTS716G
- IC4: value ST1S10PHR -> STM32F030F4P; device vreg-pulse:ST1S10PHR -> micro-stm_v3:STM32F030F4P
- OC1: value PC817 -> PC817SMD; device my_mixed:PC817 -> my_mixed:PC817SMD; MPN (none) -> PC817X2CSP9F
- Q1: value IRF7425 -> BSS138; device m-pad-2.1:IRF7425 -> m-pad-2.1:BSS138
- R1, R10, R2: value (none) -> 150
- R13: value 680 -> 22.1K; MPN (none) -> TR0805B22K1P0525Z
- R14: value 10K -> 124K; MPN (none) -> AR05BTCW1253
- R15: value 100K -> 10k
- R3: value (none) -> 10k
- R4: value (none) -> 2.2k
- R5: value 100K -> 10k; device rcl:R-EU_M0805 -> resistor:R-EU_R0805
- R6: value 20K -> 10k; device rcl:R-EU_M0805 -> resistor:R-EU_R0805
- R8: value 105K -> 10K
- R9: value (none) -> 10K; device resistor:R-EU_R0805 -> rcl:R-EU_M0805
- U$1: value GL852G-SSOP28 -> MP1584; device genesys-logic:GL852G-SSOP28 -> MP1584-dc-brick:MP1584
Connections:
- removed net +12VACC: D3.C, Q2.G, R2.2, R3.1, R4.2
- removed net +12VBATT: C12.2, C13.2, C7.2, C8.2, IC4.VIN_A, IC4.VIN_SW, IC5.VIN_A, IC5.VIN_SW, Q1.D@4
- removed net +5V: GPIO1.P
- removed net +5V2: Q7.S@3, R9.2
- removed net +BATT: D1.A
- removed net DM: GPIO3.P, U$1.DM0
- removed net DP: GPIO5.P, U$1.DP0
- removed net EN_IN: IC4.EN, IC5.EN, R18.2, R19.2
- removed net GND2: C11.1, C7.1, C8.1, IC4.AGND, IC4.H@1, IC4.H@2, IC4.H@3, IC4.H@4, IC4.H@5, IC4.H@6, IC4.PGND, IC4.SYNC, R16.2, R18.1, Z2.2
- removed net GND3: C12.1, C13.1, C14.1, IC5.AGND, IC5.H@1, IC5.H@2, IC5.H@3, IC5.H@4, IC5.H@5, IC5.H@6, IC5.PGND, IC5.SYNC, R19.1, R6.2, Z3.2
- removed net N$17: C19.2, R14.1, R15.2, U$1.!RESET
- removed net POWER_HUB: Q8.G, R10.2
- removed net VBUS: C17.2, C18.2, GPIO2.P, R14.2, U$1.V5
- removed net ПИТАНИЕ_ПК: Z2.3
- removed net ПИТАНИЕ_ХАБ: Z3.3
- new net 1WIRE: 1WIRE-1.S, IC4MCU.PA5
- new net 3V3: 3V3_1.P, GPIO27.P, GPS-4.S, I2C_VIM-4.S, I2SVIM-6.S, IC4MCU.PA1
- new net ACC: D2.A, IC4MCU.PA2, R3.1, R4.2
- new net ARDUINO_PWR: C1.2, IC1.IN, IC2G$1.OUT1
- new net BCK: 30.P, I2SVIM-3.S
- new net FAN: IC4MCU.PA7, R10.2
- new net HUB_CTRL: IC2G$1.IN4, IC4MCU.PA3
- new net HUB_PWR: IC2G$1.OUT4, U$1.VIN+
- new net I2C_SCK_A: 22.P, I2C_VIM-2.S
- new net I2C_SDA_A: 23.P, I2C_VIM-3.S
- new net I2S_LCK: 32.P, I2SVIM-5.S
- new net I2S_SCK: 29.P, I2SVIM-2.S
- new net I2S_SDO: 31.P, I2SVIM-4.S
- new net N$23: +12VSCR\.P, F3.2
- new net N$51: C16.2, U2.SS
- new net N$52: C17.2, U2.VREG5
- new net N$53: C18.1, U2.VBST
- new net N$54: C18.2, L2.1, U2.SW
- new net N$55: R13.1, R14.2, U2.VFB
- new net N$56: R15.2, U2.EN
- new net PC_CTRL: IC2G$1.IN3, IC4MCU.OSC_IN
- new net PC_PWR: C14.1, C15.2, IC2G$1.OUT3, R15.1, U2.VIN
- new net SCL: I2C-3.S, IC4MCU.PA9
- new net SCREEN_CTRL: IC2G$1.IN2, IC4MCU.OSC_OUT
- new net SCREEN_PWR: F3.1, IC2G$1.OUT2
- new net SDA: I2C-2.S, IC4MCU.PA10
- new net VBB: C3.+, C4.+, F1.2
- new net VIM_BTN: IC4MCU.PA6, R9.2
- new net VIM_PWR_CTRL: OC1.A, R9.1
- new net VOUT5V: C19.2, C5.2, FAN2-1.S, L2.2, PC_PWR-1.S, PC_PWR-2.S, R13.2
- net +ACC: now also F2.2, R3.2; no longer D2.A
- net BOOT0: now also IC4MCU.BOOT0, R8.2; no longer IC2MCU.BOOT0, R12.2
- net GND: now also 1WIRE-2.S, 28.P, C11.2, C12.2, C14.2, C15.1, C16.1, C3.-, C4.-, C5.1, C8.2, GND.P, GNDGPS.P, GNDHUB.P, GNDSCR.P, GPS-1.S, I2C-4.S, I2C_VIM-1.S, I2SVIM-1.S, OC1.C, PC_PWR-3.S, PC_PWR-4.S, PWR-2.S, Q1.S, R1.2, R14.1, R2.2, R5.2, R6.2, R8.1, SWD-4.S, U$1.VIN-, U$1.VOUT-, U2.GND, U2.PAD, USB1-4.S; no longer C10.2, C15.2, C16.2, C18.1, C20.1, C21.1, C3.1, C4.1, C5.2, C6.2, C9.2, GPIO6.P, Q2.S, Q8.S, R10.1, R12.1, R13.2, R15.1, R2.1, X1-4.S
- net N$1: now also IC2G$1.GND1/2, R1.1; no longer D1.C, Q1.S@3, R1.2
- net N$10: now also BT1.-, RTC-.P; no longer IC4.SW, L3.1
- net N$11: now also GPS-2.S, RX.P; no longer C11.2, L3.2, R17.1, Z2.1
- net N$12: now also GPS-3.S, TX.P; no longer IC5.SW, L4.1
- net N$13: now also BTN-2.S, IC4MCU.PA0-WKUP, R5.1; no longer IC4.FB, R16.1, R17.2
- net N$14: now also F2.1, PWR-3.S; no longer C14.2, L4.2, R8.1, Z3.1
- net N$15: now also BT1.+, RTC+.P; no longer IC5.FB, R6.1, R8.2
- net N$16: now also D1.A, PWR-1.S; no longer R13.1, U$1.RREF
- net N$18: now also +5VHUB.P, U$1.VOUT+; no longer C21.2, Q3.1, U$1.X2
- net N$19: now also D1.C, F1.1; no longer C20.2, Q3.2, U$1.X1
- net N$2: now also +5V.P, USB1-1.S; no longer D2.C, R3.2
- net N$3: now also FAN2-2.S, Q1.D; no longer Q7.G, Q8.D, R9.1
- net N$4: now also D2.C, D3.C, IC2G$1.IN1; no longer Q1.G, Q2.D, R1.1
- net N$5: now also IC2G$1.GND3/4, R2.1; no longer C15.1, C16.1, C5.1, L1.2, U$1.AVDD
- net N$6: now also BTN-1.S, IC4MCU.PA4, R6.1; no longer R7.1, U$1.PSELF
- net N$7: now also DM1.P, USB1-2.S; no longer C1.2, IC1.IN
- net N$8: now also DP1.P, USB1-3.S; no longer R5.1, U$1.PGANG
- net N$9: now also Q1.G, R10.1; no longer C3.2, C4.2, L1.1, R5.2, R7.2, U$1.DVDD, U$1.V33
- net NRST: now also C8.1, IC4MCU.NRST, R7.1; no longer C6.1, IC2MCU.NRST, R11.1
- net SELF_POWER: now also IC4MCU.PB1
- net SWCLK: now also IC4MCU.PA14, SWD-3.S; no longer IC2MCU.PA14, X1-3.S
- net SWIO: now also IC4MCU.PA13, SWD-2.S; no longer IC2MCU.PA13, X1-2.S
- net VDD: now also 1WIRE-3.S, BTN-3.S, C11.1, C12.1, I2C-1.S, IC1.OUT1, IC4MCU.VDDA, R7.2, SWD-1.S; no longer C10.1, C9.1, IC2MCU.VDDA, R11.2, X1-1.S
- net VIM_POWER+: now also PWR_BT+.P
- net VIM_POWER-: now also PWR_BT-.P
Other:
- moved on the sheet: C1, C11, C12, C14, C15, C16, C17, C18, C19, C2, C5, C8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

Commit message: фиксы схемы
R9 FROM 10K TO 120Ohm
SWAP R13 and R14 nominal
Parts:
- R13: value 22.1K -> 124K
- R14: value 124K -> 22.1К
- R9: value 10K -> 120
Other:
- note added: "1.0 - INITIAL RELEASE 1.1 - FIXED R9 FROM 10K TO 120Ohm SWAP R13 and R14 nominal"
Changed lines of the file:
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@@
 <?xml version="1.0" encoding="utf-8"?>
 <!DOCTYPE eagle SYSTEM "eagle.dtd">
-<eagle version="9.3.0">
+<eagle version="9.5.2">
 <drawing>
 <settings>
@@
 <part name="+5VHUB" library="wirepad" library_urn="urn:adsk.eagle:library:412" deviceset="1,6/0,8" device="" package3d_urn="urn:adsk.eagle:package:30830/1"/>
 <part name="GNDHUB" library="wirepad" library_urn="urn:adsk.eagle:library:412" deviceset="1,6/0,8" device="" package3d_urn="urn:adsk.eagle:package:30830/1"/>
-<part name="R9" library="rcl" library_urn="urn:adsk.eagle:library:334" deviceset="R-EU_" device="M0805" package3d_urn="urn:adsk.eagle:package:23556/2" value="10K"/>
+<part name="R9" library="rcl" library_urn="urn:adsk.eagle:library:334" deviceset="R-EU_" device="M0805" package3d_urn="urn:adsk.eagle:package:23556/2" value="120"/>
 <part name="I2C" library="con-molex" library_urn="urn:adsk.eagle:library:165" deviceset="53?-04" device="047" package3d_urn="urn:adsk.eagle:package:8078513/1" value="i2c"/>
 <part name="FAN2" library="con-molex" library_urn="urn:adsk.eagle:library:165" deviceset="53?-02" device="047" package3d_urn="urn:adsk.eagle:package:8078511/1"/>
@@
 <attribute name="MPN" value="CL31A476MPHNNNE"/>
 </part>
-<part name="R13" library="rcl" library_urn="urn:adsk.eagle:library:334" deviceset="R-EU_" device="M0805" package3d_urn="urn:adsk.eagle:package:23556/2" value="22.1K">
+<part name="R13" library="rcl" library_urn="urn:adsk.eagle:library:334" deviceset="R-EU_" device="M0805" package3d_urn="urn:adsk.eagle:package:23556/2" value="124K">
 <attribute name="MPN" value="TR0805B22K1P0525Z"/>
 </part>
-<part name="R14" library="rcl" library_urn="urn:adsk.eagle:library:334" deviceset="R-EU_" device="M0805" package3d_urn="urn:adsk.eagle:package:23556/2" value="124K">
+<part name="R14" library="rcl" library_urn="urn:adsk.eagle:library:334" deviceset="R-EU_" device="M0805" package3d_urn="urn:adsk.eagle:package:23556/2" value="22.1К">
 <attribute name="MPN" value="AR05BTCW1253"/>
 </part>
@@
 <sheet>
 <plain>
-<text x="123.19" y="128.27" size="1.778" layer="91">R1 = R2 x (VOUT - VFB) / VFB</text>
+<text x="138.43" y="158.75" size="1.778" layer="91">R1 = R2 x (VOUT - VFB) / VFB</text>
+<text x="139.7" y="149.86" size="1.778" layer="91">1.0 - INITIAL RELEASE
+1.1 - FIXED R9 FROM 10K TO 120Ohm
+        SWAP R13 and R14 nominal</text>
 </plain>
 <instances>
@@
 </drawing>
 <compatibility>
+<note version="6.3" minversion="6.2.2" severity="warning">
+Since Version 6.2.2 text objects can contain more than one line,
+which will not be processed correctly with this version.
+</note>
 <note version="8.2" severity="warning">
 Since Version 8.2, EAGLE supports online libraries. The ids
